File: PCB/CycloRadarDemoKit/CycloRadarDemoKit.kicad_sch (KiCad schematic)
At the start: 18 parts, among them J101 JTAG, SW101 RESET, SW102 BOOT MODE, U101 ESP32-WROVER-E

Commit message: RJ45 chose, leds connected
Parts:
- C102, C103: value 1uF/16V(10%) -> 1uF/50V(10%); footprint (none) -> Capacitor_SMD:C_0603_1608Metric; LCSC (none) -> C15849
- C104: value 0.1uF/16V(10%) -> 0.1uF/50V(10%); footprint (none) -> Capacitor_SMD:C_0603_1608Metric; LCSC (none) -> C14663
- D101, D102: LCSC (none) -> C283256
- R104, R105, R106: footprint (none) -> Resistor_SMD:R_0805_2012Metric; LCSC (none) -> C17477
- SW101, SW102: footprint (none) -> Button_Switch_SMD:SW_SPST_TS-1088R; LCSC (none) -> C455280
- U101: LCSC (none) -> C529589
Other:
- note added: "Q: MLCC 100uF is not available, can I use electrolytic or tantal?"
- note added: "TODO: Choose RC and Ferrite B. components on JLC"
Changed lines of the file:
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@@
     (stroke (width 0) (type default))
+  )
+  (text "TODO: Choose RC and Ferrite B. components on JLC" (at 104.14 111.76 0)
+    (effects (font (size 1.27 1.27)) (justify left bottom))
   )
   (text "Some GPIO" (at 224.79 149.86 0)
@@
   (text "Strapping pins:\nMTDI(IO12) - LDO voltage setting (0)\nIO0 - Boot (SPI, UART) (1)\nIO2 - Boot (SPI, UART) (0)\nMTDO(IO15) - debug log on boot (1)\nIO5 - SDIO function (1)\n\nInternal flash pins:\n17-22\n\nAll GND symbols refer to same ground\n"
     (at 241.3 40.64 0)
+    (effects (font (size 1.27 1.27)) (justify left bottom))
+  )
+  (text "Q: MLCC 100uF is not available, can I use electrolytic or tantal?"
+    (at 60.96 25.4 0)
     (effects (font (size 1.27 1.27)) (justify left bottom))
   )
@@
       (effects (font (size 1.27 1.27)))
     )
-    (property "Footprint" "" (at 31.75 165.1 0)
+    (property "Footprint" "Button_Switch_SMD:SW_SPST_TS-1088R" (at 31.75 165.1 0)
       (effects (font (size 1.27 1.27)) hide)
     )
     (property "Datasheet" "~" (at 31.75 165.1 0)
+      (effects (font (size 1.27 1.27)) hide)
+    )
+    (property "LCSC" "C455280" (at 31.75 170.18 0)
       (effects (font (size 1.27 1.27)) hide)
     )
@@
       (effects (font (size 1.27 1.27)) (justify left))
     )
-    (property "Value" "1uF/16V(10%)" (at 110.49 35.5663 0)
-      (effects (font (size 1.27 1.27)) (justify left))
-    )
-    (property "Footprint" "" (at 107.95 34.29 0)
+    (property "Value" "1uF/50V(10%)" (at 110.49 35.5663 0)
+      (effects (font (size 1.27 1.27)) (justify left))
+    )
+    (property "Footprint" "Capacitor_SMD:C_0603_1608Metric" (at 107.95 34.29 0)
       (effects (font (size 1.27 1.27)) hide)
     )
     (property "Datasheet" "~" (at 107.95 34.29 0)
+      (effects (font (size 1.27 1.27)) hide)
+    )
+    (property "LCSC" "C15849" (at 107.95 34.29 0)
       (effects (font (size 1.27 1.27)) hide)
     )
@@
       (effects (font (size 1.27 1.27)) (justify left) hide)
     )
-    (property "Datasheet" "http://www.diodes.com/_files/datasheets/ds11005.pdf" (at 68.58 161.29 0)
+    (property "Datasheet" "https://datasheet.lcsc.com/lcsc/2304140030_STMicroelectronics-BAT54AFILM_C283256.pdf" (at 68.58 161.29 0)
+      (effects (font (size 1.27 1.27)) hide)
+    )
+    (property "LCSC" "C283256" (at 72.39 171.45 0)
       (effects (font (size 1.27 1.27)) hide)
     )
@@
     )
     (property "Datasheet" "https://www.espressif.com/sites/default/files/documentation/esp32-wrover-e_esp32-wrover-ie_datasheet_en.pdf" (at 134.62 101.6 0)
+      (effects (font (size 1.27 1.27)) hide)
+    )
+    (property "LCSC" "C529589" (at 132.08 66.04 0)
       (effects (font (size 1.27 1.27)) hide)
     )
@@
       (effects (font (size 1.27 1.27)) (justify left))
     )
-    (property "Value" "0.1uF/16V(10%)" (at 43.18 156.2163 0)
-      (effects (font (size 1.27 1.27)) (justify left))
-    )
-    (property "Footprint" "" (at 45.72 154.94 0)
+    (property "Value" "0.1uF/50V(10%)" (at 43.18 156.2163 0)
+      (effects (font (size 1.27 1.27)) (justify left))
+    )
+    (property "Footprint" "Capacitor_SMD:C_0603_1608Metric" (at 45.72 154.94 0)
       (effects (font (size 1.27 1.27)) hide)
     )
     (property "Datasheet" "~" (at 45.72 154.94 0)
+      (effects (font (size 1.27 1.27)) hide)
+    )
+    (property "LCSC" "C14663" (at 45.72 154.94 0)
       (effects (font (size 1.27 1.27)) hide)
     )
@@
       (effects (font (size 1.27 1.27)))
     )
-    (property "Footprint" "" (at 69.85 119.888 90)
+    (property "Footprint" "Resistor_SMD:R_0805_2012Metric" (at 69.85 119.888 90)
       (effects (font (size 1.27 1.27)) hide)
     )
     (property "Datasheet" "~" (at 69.85 118.11 0)
+      (effects (font (size 1.27 1.27)) hide)
+    )
+    (property "LCSC" "C17477" (at 69.85 118.11 0)
       (effects (font (size 1.27 1.27)) hide)
     )
@@
       (effects (font (size 1.27 1.27)) (justify left) hide)
     )
-    (property "Datasheet" "http://www.diodes.com/_files/datasheets/ds11005.pdf" (at 68.58 142.24 0)
+    (property "Datasheet" "https://datasheet.lcsc.com/lcsc/2304140030_STMicroelectronics-BAT54AFILM_C283256.pdf" (at 68.58 142.24 0)
+      (effects (font (size 1.27 1.27)) hide)
+    )
+    (property "LCSC" "C283256" (at 72.39 152.4 0)
       (effects (font (size 1.27 1.27)) hide)
     )
@@
       (effects (font (size 1.27 1.27)))
     )
-    (property "Footprint" "" (at 217.17 151.638 90)
+    (property "Footprint" "Resistor_SMD:R_0805_2012Metric" (at 217.17 151.638 90)
       (effects (font (size 1.27 1.27)) hide)
     )
@@
       (effects (font (size 1.27 1.27)) hide)
     )
+    (property "LCSC" "C17477" (at 217.17 149.86 0)
+      (effects (font (size 1.27 1.27)) hide)
+    )
     (pin "2")
     (pin "1")
@@
       (effects (font (size 1.27 1.27)))
     )
-    (property "Footprint" "" (at 31.75 146.05 0)
+    (property "Footprint" "Button_Switch_SMD:SW_SPST_TS-1088R" (at 31.75 146.05 0)
       (effects (font (size 1.27 1.27)) hide)
     )
@@
       (effects (font (size 1.27 1.27)) hide)
     )
+    (property "LCSC" "C455280" (at 31.75 151.13 0)
+      (effects (font (size 1.27 1.27)) hide)
+    )
     (pin "1")
     (pin "2")
@@
       (effects (font (size 1.27 1.27)) (justify left))
     )
-    (property "Value" "1uF/16V(10%)" (at 77.47 52.0763 0)
-      (effects (font (size 1.27 1.27)) (justify left))
-    )
-    (property "Footprint" "" (at 74.93 50.8 0)
+    (property "Value" "1uF/50V(10%)" (at 77.47 52.0763 0)
+      (effects (font (size 1.27 1.27)) (justify left))
+    )
+    (property "Footprint" "Capacitor_SMD:C_0603_1608Metric" (at 74.93 50.8 0)
       (effects (font (size 1.27 1.27)) hide)
     )
     (property "Datasheet" "~" (at 74.93 50.8 0)
+      (effects (font (size 1.27 1.27)) hide)
+    )
+    (property "LCSC" "C15849" (at 74.93 50.8 0)
       (effects (font (size 1.27 1.27)) hide)
     )
@@
       (effects (font (size 1.27 1.27)))
     )
-    (property "Footprint" "" (at 69.85 118.872 90)
+    (property "Footprint" "Resistor_SMD:R_0805_2012Metric" (at 69.85 118.872 90)
       (effects (font (size 1.27 1.27)) hide)
     )
@@
       (effects (font (size 1.27 1.27)) hide)
     )
+    (property "LCSC" "C17477" (at 69.85 120.65 0)
+      (effects (font (size 1.27 1.27)) hide)
+    )

Commit message: RJ45 footprint added
Connections:
- net IO0 is gone; now on net MAC_CLK: D102.3
Other:
- note added: "IO0"
Changed lines of the file:
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@@
-    (stroke (width 0) (type default))
-  )
-  (wire (pts (xy 80.01 173.99) (xy 83.82 173.99))
     (stroke (width 0) (type default))
   )
@@
     (stroke (width 0) (type default))
   )
+  (wire (pts (xy 93.98 173.99) (xy 80.01 173.99))
+    (stroke (width 0) (type default))
+  )
   (wire (pts (xy 73.66 120.65) (xy 82.55 120.65))
     (stroke (width 0) (type default))
@@
   (text "TODO: Choose RC and Ferrite B. components on JLC" (at 104.14 111.76 0)
     (effects (font (size 1.27 1.27)) (justify left bottom))
+  )
+  (text "IO0" (at 80.01 173.99 0)
+    (effects (font (size 1.27 1.27) (color 0 0 0 1)) (justify left bottom))
   )
   (text "Some GPIO" (at 224.79 149.86 0)
@@
     (effects (font (size 1.27 1.27)) (justify left bottom))
   )
-  (label "IO0" (at 83.82 173.99 180) (fields_autoplaced)
-    (effects (font (size 1.27 1.27)) (justify right bottom))
-  )
   (label "MAC_MDC" (at 182.88 76.2 180) (fields_autoplaced)
     (effects (font (size 1.27 1.27)) (justify right bottom))
@@
     (effects (font (size 1.27 1.27)) (justify left bottom))
   )
+  (label "MAC_CLK" (at 93.98 173.99 180) (fields_autoplaced)
+    (effects (font (size 1.27 1.27)) (justify right bottom))
+  )
   (label "+3V3" (at 190.5 139.7 180) (fields_autoplaced)

Commit message: MCU routed, two GPIO tested
Parts:
- added R108: 10K(5%), symbol Device:R
Connections:
- net +3V3: now also R108.2
- net GPIO2: now also R106.2
- net LED_DIN: now reaches U101.26 (ADC2_CH0/GPIO4)
- net Photo_res: now reaches U101.4 (SENSOR_VP/GPIO36/ADC1_CH0)
- net IMU_INT: now reaches U101.5 (SENSOR_VN/GPIO39/ADC1_CH3)
- net SDA: now reaches U101.6 (GPIO34/ADC1_CH6)
- net SCL: now reaches U101.7 (GPIO35/ADC1_CH7)
- net PMIC_INT: now reaches U101.8 (32K_XP/GPIO32/ADC1_CH4)
- net 12V_DIS: now reaches U101.9 (32K_XN/GPIO33/ADC1_CH5)
- net 12V_DIS: now also R108.1
Other:
- sheet IMU&ANT renamed IMU + ANT
- sheet USB interface renamed USB + LED
- sheet Power management ports: added 12V_DIS; removed 12V_EN
- note added: "!!! TODO: Chech the GPIO purpose: GPIO for I2C GPIO for INT GPIO for ADC GPIO 4 LED OK GPIO 33 OK"
- note added: "Global I2C bus: IMU A IMU B Power monitor EXT dev"
- note added: "Global power rails"
- note added: "Strapping pins: (default) MTDI(IO12) - LDO voltage setting (0) IO0 - Boot (SPI, UART) (1) IO2 - Boot (SPI, UART) (0) MTDO(IO15) - debug log on boot (1) IO5 - SDIO function (1) Internal flash pins: 17-22 All GND symbols refer to same ground"
- note added: "TODO: Expose I2C pins to piheader"
- note added: "Versatile GPIO (it's also bootstrap pin)"
- note removed: "Some GPIO"
- note removed: "Strapping pins: MTDI(IO12) - LDO voltage setting (0) IO0 - Boot (SPI, UART) (1) IO2 - Boot (SPI, UART) (0) MTDO(IO15) - debug log on boot (1) IO5 - SDIO function (1) Internal flash pins: 17-22 All GND symbols refer to same ground"
- moved on the sheet: C101, C102, C103, C104, D101, D102, R102, R104, R105, R107, SW101, SW102
