File: PCB/CycloRadarDemoKit/CycloRadarDemoKit.kicad_sch (KiCad schematic)
At the start: 12 parts, among them J101 I2C conn, J102 CAN, J103 100BASE-T1, J104 Radar debug, U101 RADAR POGO pins

Commit message: PCB edited, 3D case mock-up
Parts:
- added J105: Radar pins, Connector_PinHeader_1.27mm:PinHeader_1x10_P1.27mm_Vertical, symbol Connector_Generic:Conn_01x10
Connections:
- net +12V: now also J105.10 (Pin_10); no longer U101.1 (Pin_1)
- net CANH: now also J105.2 (Pin_2); no longer U101.9 (Pin_9)
- net CANL: now also J105.1 (Pin_1); no longer U101.10 (Pin_10)
- net ETH_H: now also J105.4 (Pin_4); no longer U101.7 (Pin_7)
- net ETH_L: now also J105.3 (Pin_3); no longer U101.8 (Pin_8)
- net GND: now also J105.5 (Pin_5); no longer U101.6 (Pin_6)
- net MID1: now also J105.9 (Pin_9); no longer U101.2 (Pin_2)
- net MID2: now also J105.8 (Pin_8); no longer U101.3 (Pin_3)
- net MID3: now also J105.7 (Pin_7); no longer U101.4 (Pin_4)
- net MID4: now also J105.6 (Pin_6); no longer U101.5 (Pin_5)
Other:
- moved on the sheet: U101
Changed lines of the file:
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@@
+    )
+  )
+  (symbol (lib_id "Connector_Generic:Conn_01x10") (at 251.46 71.12 0) (unit 1)
+    (in_bom yes) (on_board yes) (dnp no) (fields_autoplaced)
+    (property "Reference" "J105" (at 254 71.12 0)
+      (effects (font (size 1.27 1.27)) (justify left))
+    )
+    (property "Value" "Radar pins" (at 254 73.66 0)
+      (effects (font (size 1.27 1.27)) (justify left))
+    )
+    (property "Footprint" "Connector_PinHeader_1.27mm:PinHeader_1x10_P1.27mm_Vertical" (at 251.46 71.12 0)
+      (effects (font (size 1.27 1.27)) hide)
+    )
+    (property "Datasheet" "~" (at 251.46 71.12 0)
+      (effects (font (size 1.27 1.27)) hide)
+    )
+    (pin "1")
+    (pin "2")
+    (pin "6")
+    (pin "7")
+    (pin "4")
+    (pin "8")
+    (pin "9")
+    (pin "10")
+    (pin "3")
+    (pin "5")
+    (instances
+      (project "CycloRadarDemoKit"
+        (path "/c2cd7ca4-4652-4b3d-a3a8-1cfa66cb11e9"
+          (reference "J105") (unit 1)
+        )
+      )
     )
   )
@@
     )
   )
-  (symbol (lib_id "alps_modules:ALPS_Generic_Radar_5") (at 251.46 72.39 180) (unit 1)
+  (symbol (lib_id "alps_modules:ALPS_Generic_Radar_5") (at 271.78 72.39 180) (unit 1)
     (in_bom yes) (on_board yes) (dnp no) (fields_autoplaced)
-    (property "Reference" "U101" (at 254 71.12 0)
+    (property "Reference" "U101" (at 274.32 71.12 0)
       (effects (font (size 1.27 1.27)) (justify right))
     )
-    (property "Value" "RADAR POGO pins" (at 254 73.66 0)
+    (property "Value" "RADAR POGO pins" (at 274.32 73.66 0)
       (effects (font (size 1.27 1.27)) (justify right))
     )
-    (property "Footprint" "alps_modules:ALPS_USRR5" (at 251.46 72.39 0)
+    (property "Footprint" "alps_modules:ALPS_USRR5" (at 271.78 72.39 0)
       (effects (font (size 1.27 1.27)) hide)
     )
-    (property "Datasheet" "" (at 251.46 72.39 0)
+    (property "Datasheet" "" (at 271.78 72.39 0)
       (effects (font (size 1.27 1.27)) hide)
     )
