File: PCB/CycloRadarDemoKit/CycloRadarDemoKit.kicad_pcb (KiCad board)
At the start: 4 copper layers, 58.8 x 117.8 mm, 171 parts, among them J101 I2C conn, J102 CAN, J103 100BASE-T1, J104 Radar debug, J201 ARJM11B1-009-AB-EW2, J301 USB_C_Receptacle_USB2.0, J401 20-16V Supply Voltage, J501 ANT_JTAG, Q301 L8050QLT1G, Q302 L8050QLT1G, Q401 SI2309CDS, Q601 L8050QLT1G, SW801 RESET, SW802 BOOT MODE, U101 RADAR POGO pins, U201 IP101GRI, U301 CP2102N-Axx-xQFN24, U401 INA3221, U402 RT8259, U403 AP63205WU, U501 D52MxxM8, U502 MPU-6050, U701 TPS2121RUXR, U702 AP63203WU, U801 ESP32-WROVER-E-N16R8, Y201 25MHz

Commit message: PCB mockup, grid repaired
Parts:
- J201: footprint Connector_RJ:CONN_JXD2-0Z10NL_PUL -> Connector_RJ:CONN12_5-2301995-3_TEC
- moved R215 148.5 mm to (28.4, 22.5)
- moved C210 116.1 mm to (106.8, 47.2)
- moved D616 81.9 mm to (98.3, 88.6)
- moved D614 54.3 mm to (228.5, 144.8)
- moved D606 37.6 mm to (210.8, 40.0)
- moved D607 37.6 mm to (217.8, 40.0)
- moved D604 24.7 mm to (172.3, 44.5)
- moved D605 17.1 mm to (183.3, 44.5)
- moved D609 16.9 mm to (201.8, 75.0)
- moved D615 16.3 mm to (132.3, 158.4)
- moved D617 14.3 mm to (147.3, 158.4)
- moved D620 9.55 mm to (131.3, 68.5)
- moved D621 5.10 mm to (130.3, 53.0)
- moved D613 4.95 mm to (167.8, 158.4)
- moved D603 3.96 mm to (142.3, 44.5)
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Other:
- board size 58.8 x 117.8 mm -> 60 x 120 mm

Commit message: layout mockup done
Parts:
- removed the D607 at (217.8, 40.0)
- removed the D614 at (228.5, 144.8)
- removed the D616 at (98.3, 88.6)
- removed D618, D619, D620, D621: WS2812B, LED_SMD:LED_SK6812MINI_PLCC4_3.5x3.5mm_P1.75mm
- removed the R406 at (173.8, 22.4)
- added D605: WS2812B, LED_SMD:LED_SK6812MINI_PLCC4_3.5x3.5mm_P1.75mm, F.Cu at (130.1, 58.5)
- added D613: WS2812B, LED_SMD:LED_SK6812MINI_PLCC4_3.5x3.5mm_P1.75mm, F.Cu at (130.1, 74.5)
- added D615: WS2812B, LED_SMD:LED_SK6812MINI_PLCC4_3.5x3.5mm_P1.75mm, F.Cu at (130.1, 144.4)
- R407: footprint Resistor_SMD:R_0805_2012Metric -> Resistor_SMD:R_1210_3225Metric
- TP201, TP202, TP203, TP501, TP502, TP503: footprint TestPoint:TestPoint_Pad_D2.0mm -> TestPoint:TestPoint_Pad_D1.0mm
- moved R602 199.4 mm to (184.8, 64.2)
- moved R603 199.4 mm to (184.8, 66.7)
- moved R604 199.4 mm to (184.8, 69.2)
- moved D617 193.4 mm to (180.1, 63.5)
- moved R202 189.8 mm to (161.5, 74.5)
- moved R206 189.8 mm to (161.5, 72.0)
- moved R205 189.5 mm to (161.7, 70.0)
- moved R203 189.5 mm to (161.5, 77.4)
- moved R204 189.5 mm to (161.5, 80.0)
- moved R209 189.3 mm to (161.2, 82.5)
- moved Q601 186.5 mm to (179.2, 59.4)
- moved R212 181.2 mm to (152.6, 81.5)
- moved JP501 180.8 mm to (164.3, 151.9), turned to 90 degrees
- moved TP201 176.3 mm to (165.3, 69.7)
- moved TP203 176.0 mm to (165.3, 72.0)
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- renumbered D602 to D601, D603 to D602, D604 to D603, D605 to D604, D608 to D607, D609 to D608, D610 to D609, D611 to D610, D612 to D611, D613 to D612, D615 to D614, D617 to D616, D601 to D617
Connections:
- D604 pad 2: Net-(D605-DOUT) -> Net-(D604-DOUT)
- D607 pad 4: Net-(D607-DOUT) (its old number) -> Net-(D606-DOUT)
- D616 pad 2: Net-(D617-DOUT) -> unconnected-(D616-DOUT-Pad2)
- J201 pad 13: (no net) -> unconnected-(J201-NC-Pad13)
- J201 pad 14: (no net) -> unconnected-(J201-NC-Pad14)
- J201 pad P1: (no net) -> /PHY/TD+
- J201 pad P2: (no net) -> /PHY/TD-
- J201 pad P3: (no net) -> /PHY/RD+
- J201 pad P4: (no net) -> Net-(J201-RCT)
- J201 pad P5: (no net) -> Net-(J201-RCT)
- J201 pad P6: (no net) -> /PHY/RD-
- J201 pad P7: (no net) -> unconnected-(J201-NC-PadP7)
- J201 pad P8: (no net) -> Net-(C212-Pad1)
- R402 pad 2: Net-(R402-Pad2) -> Net-(Q401-S)
- R403 pad 2: Net-(R403-Pad2) -> Net-(U402-VIN)
- R404 pad 2: Net-(R404-Pad2) -> Net-(C404-Pad2)
- R406 pad 2: Net-(R403-Pad2) -> Net-(U402-VIN)
- R408 pad 1: Net-(R407-Pad2) -> Net-(R405-Pad2)
Other:
- outline, holes or cut-outs redrawn

Commit message: PCB, 3Dmodel
mockup PCB version done, schcematic exported to latex, 3D model generated and exported to latex
Parts:
- moved R808 23.7 mm to (155.8, 64.3), turned to 0 degrees
- moved R807 21.8 mm to (156.0, 61.6), turned to 0 degrees
- moved TP501 21.5 mm to (121.0, 137.6)
- moved TP502 21.5 mm to (121.0, 142.6)
- moved R503 20.8 mm to (135.3, 138.3)
- moved R806 20.6 mm to (156.0, 59.1), turned to 0 degrees
- moved R702 19.9 mm to (135.3, 95.6)
- moved R805 19.8 mm to (156.0, 56.6), turned to 0 degrees
- moved J501 19.7 mm to (129.6, 140.3)
- moved C301 19.0 mm to (124.9, 90.5)
- moved C302 19.0 mm to (124.9, 93.5)
- moved R308 18.8 mm to (129.2, 97.2)
- moved R301 18.8 mm to (125.1, 97.1)
- moved FB501 18.8 mm to (138.6, 85.6)
- moved R307 18.6 mm to (122.8, 117.8)
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Other:
- board text added: "100BASE-T1"
- board text added: "20-16V Supply Voltage"
- board text added: "ESP32"
- board text added: "Ethernet"
- board text added: "I2C"
- board text added: "JTAG"
- board text added: "RSS DEMO module (mock-up)"
- board text added: "Radar debug"
- board text added: "USB"
- board text removed: "THT connectors are on the back side!!!"
- board text removed: "TODO: Consider 0402!!!"
- board text removed: "TODO: Double side assembly!!!"
- board text removed: "TODO: IP101 clearence problem!!!"
- board text removed: "TODO: Length matching on RMII"
- board text removed: "X = 55mm Y = 55mm"
