File: PCB/CycloRadarDemoKit/Power_2.kicad_sch (KiCad schematic)
At the start: 16 parts, among them U401 AP63203WU, U404 TPS2121RUXR

Commit message: photos added, readme rewrited
Parts:
- renumbered C410 to C801, C401 to C802, C402 to C803, C708 to C804, C404 to C805, D401 to D801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
